File: SingleESC.sch (KiCad schematic (older format))
At the start: 32 parts, among them P19 Pad, P3 Pad, P4 Pad, P5 Pad, P6 Pad, Q1 NTLUD4C26N, Q2 NTLUD4C26N, Q3 NTLUD4C26N, U3 EFM8BB21-QFN20, U4 TPS51604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

Commit message: Finished Routing
Parts:
- added P23, P24: Pad, custom:FlashPad, symbol 6sESC:Pad
Connections:
- wire segments 174 -> 177
- no-connect marks 9 -> 8
Changed lines of the file:
@@
 AR Path="/5A7C7635/5A8007A7" Ref="U12"  Part="1"
 AR Path="/5A7C8234/5A8007A7" Ref="U16"  Part="1"
-F 0 "U16" H 6400 2137 60  0000 C CNN
+F 0 "U4" H 6400 2137 60  0000 C CNN
 F 1 "TPS51604" H 6400 2031 60  0000 C CNN
 F 2 "custom:8-WFDFN" H 6400 1600 60  0001 C CNN
@@
 AR Path="/5A7C7635/5A8007AE" Ref="U11"  Part="1"
 AR Path="/5A7C8234/5A8007AE" Ref="U15"  Part="1"
-F 0 "U15" H 3200 4050 60  0000 C CNN
+F 0 "U3" H 3200 4050 60  0000 C CNN
 F 1 "EFM8BB21-QFN20" H 3200 3944 60  0000 C CNN
 F 2 "custom:QFN20" H 3200 3200 60  0001 C CNN
@@
 AR Path="/5A7C7635/5A8007D3" Ref="C24"  Part="1"
 AR Path="/5A7C8234/5A8007D3" Ref="C32"  Part="1"
-F 0 "C32" V 6148 2150 50  0000 C CNN
+F 0 "C8" V 6148 2150 50  0000 C CNN
 F 1 "1uF" V 6239 2150 50  0000 C CNN
 F 2 "custom:C_0402" H 6438 2000 50  0001 C CNN
@@
 AR Path="/5A7C7635/5A8007DC" Ref="C23"  Part="1"
 AR Path="/5A7C8234/5A8007DC" Ref="C31"  Part="1"
-F 0 "C31" V 5848 800 50  0000 C CNN
+F 0 "C7" V 5848 800 50  0000 C CNN
 F 1 "1uF" V 5939 800 50  0000 C CNN
 F 2 "custom:C_0402" H 6138 650 50  0001 C CNN
@@
 AR Path="/5A7C7635/5A8007E3" Ref="R22"  Part="1"
 AR Path="/5A7C8234/5A8007E3" Ref="R32"  Part="1"
-F 0 "R32" V 6593 800 50  0000 C CNN
+F 0 "R2" V 6593 800 50  0000 C CNN
 F 1 "3" V 6684 800 50  0000 C CNN
 F 2 "custom:R_0402" V 6730 800 50  0001 C CNN
@@
 AR Path="/5A7C7635/5A8007EA" Ref="C22"  Part="1"
 AR Path="/5A7C8234/5A8007EA" Ref="C30"  Part="1"
-F 0 "C30" V 1698 3350 50  0000 C CNN
+F 0 "C6" V 1698 3350 50  0000 C CNN
 F 1 "4.7uF" V 1789 3350 50  0000 C CNN
 F 2 "custom:C_0402" H 1988 3200 50  0001 C CNN
@@
 AR Path="/5A7C7635/5A8007FA" Ref="R21"  Part="1"
 AR Path="/5A7C8234/5A8007FA" Ref="R31"  Part="1"
-F 0 "R31" V 1743 3950 50  0000 C CNN
+F 0 "R1" V 1743 3950 50  0000 C CNN
 F 1 "1k" V 1834 3950 50  0000 C CNN
 F 2 "custom:R_0402" V 1880 3950 50  0001 C CNN
@@
 AR Path="/5A7C7635/5A800824" Ref="R25"  Part="1"
 AR Path="/5A7C8234/5A800824" Ref="R35"  Part="1"
-F 0 "R35" H 8620 1996 50  0000 L CNN
+F 0 "R5" H 8620 1996 50  0000 L CNN
 F 1 "10k" H 8620 1905 50  0000 L CNN
 F 2 "custom:R_0402" V 8480 1950 50  0001 C CNN
@@
 AR Path="/5A7C7635/5A80082B" Ref="R28"  Part="1"
 AR Path="/5A7C8234/5A80082B" Ref="R38"  Part="1"
-F 0 "R38" H 8870 1746 50  0000 L CNN
+F 0 "R8" H 8870 1746 50  0000 L CNN
 F 1 "100k" H 8870 1655 50  0000 L CNN
 F 2 "custom:R_0402" V 8730 1700 50  0001 C CNN
@@
 AR Path="/5A7C7635/5A8008AE" Ref="P12"  Part="1"
 AR Path="/5A7C8234/5A8008AE" Ref="P16"  Part="1"
-F 0 "P16" H 9378 1450 60  0000 L CNN
+F 0 "P4" H 9378 1450 60  0000 L CNN
 F 1 "Pad" H 9250 1200 60  0001 C CNN
 F 2 "custom:PhasePad" H 9250 1450 60  0001 C CNN
@@
 	3050 1700 3050 2550
 Wire Wire Line
-	3350 1700 3350 2550
+	3350 1700 3350 2300
 Wire Wire Line
 	3050 4250 3050 3850
@@
 AR Path="/5A7C7635/5A8008C3" Ref="P11"  Part="1"
 AR Path="/5A7C8234/5A8008C3" Ref="P15"  Part="1"
-F 0 "P15" H 4928 3050 60  0000 L CNN
+F 0 "P3" H 4928 3050 60  0000 L CNN
 F 1 "Pad" H 4800 2800 60  0001 C CNN
 F 2 "custom:RCPad" H 4800 3050 60  0001 C CNN
@@
 LOW_C
 NoConn ~ 2450 3450
-NoConn ~ 3250 2550
 $Comp
 L 6sESC:NTLUD4C26N Q1
@@
 AR Path="/5A7C7635/5A827F39" Ref="Q7"  Part="1"
 AR Path="/5A7C8234/5A827F39" Ref="Q10"  Part="1"
-F 0 "Q10" H 7950 1235 50  0000 C CNN
+F 0 "Q1" H 7950 1235 50  0000 C CNN
 F 1 "NTLUD4C26N" H 7950 1326 50  0000 C CNN
 F 2 "custom:UDFN6-NTLUD4" H 7950 1500 50  0001 C CNN
@@
 AR Path="/5A7C7635/5A882B6E" Ref="U13"  Part="1"
 AR Path="/5A7C8234/5A882B6E" Ref="U17"  Part="1"
-F 0 "U17" H 6450 3937 60  0000 C CNN
+F 0 "U5" H 6450 3937 60  0000 C CNN
 F 1 "TPS51604" H 6450 3831 60  0000 C CNN
 F 2 "custom:8-WFDFN" H 6450 3400 60  0001 C CNN
@@
 AR Path="/5A7C7635/5A882B75" Ref="C26"  Part="1"
 AR Path="/5A7C8234/5A882B75" Ref="C34"  Part="1"
-F 0 "C34" V 6198 3950 50  0000 C CNN
+F 0 "C10" V 6198 3950 50  0000 C CNN
 F 1 "1uF" V 6289 3950 50  0000 C CNN
 F 2 "custom:C_0402" H 6488 3800 50  0001 C CNN
@@
 AR Path="/5A7C7635/5A882B7C" Ref="C25"  Part="1"
 AR Path="/5A7C8234/5A882B7C" Ref="C33"  Part="1"
-F 0 "C33" V 5848 2600 50  0000 C CNN
+F 0 "C9" V 5848 2600 50  0000 C CNN
 F 1 "1uF" V 5939 2600 50  0000 C CNN
 F 2 "custom:C_0402" H 6138 2450 50  0001 C CNN
@@
 AR Path="/5A7C7635/5A882B83" Ref="R23"  Part="1"
 AR Path="/5A7C8234/5A882B83" Ref="R33"  Part="1"
-F 0 "R33" V 6643 2600 50  0000 C CNN
+F 0 "R3" V 6643 2600 50  0000 C CNN
 F 1 "3" V 6734 2600 50  0000 C CNN
 F 2 "custom:R_0402" V 6780 2600 50  0001 C CNN
@@
 AR Path="/5A7C7635/5A882B8A" Ref="R26"  Part="1"
 AR Path="/5A7C8234/5A882B8A" Ref="R36"  Part="1"
-F 0 "R36" H 8670 3796 50  0000 L CNN
+F 0 "R6" H 8670 3796 50  0000 L CNN
 F 1 "10k" H 8670 3705 50  0000 L CNN
 F 2 "custom:R_0402" V 8530 3750 50  0001 C CNN
@@
 AR Path="/5A7C7635/5A882B91" Ref="R29"  Part="1"
 AR Path="/5A7C8234/5A882B91" Ref="R39"  Part="1"
-F 0 "R39" H 8920 3546 50  0000 L CNN
+F 0 "R9" H 8920 3546 50  0000 L CNN
 F 1 "100k" H 8920 3455 50  0000 L CNN
 F 2 "custom:R_0402" V 8780 3500 50  0001 C CNN
@@
 AR Path="/5A7C7635/5A882B99" Ref="P13"  Part="1"
 AR Path="/5A7C8234/5A882B99" Ref="P17"  Part="1"
-F 0 "P17" H 9428 3250 60  0000 L CNN
+F 0 "P5" H 9428 3250 60  0000 L CNN
 F 1 "Pad" H 9300 3000 60  0001 C CNN
 F 2 "custom:PhasePad" H 9300 3250 60  0001 C CNN
@@
 AR Path="/5A7C7635/5A882BCE" Ref="Q8"  Part="1"
 AR Path="/5A7C8234/5A882BCE" Ref="Q11"  Part="1"
-F 0 "Q11" H 8000 3035 50  0000 C CNN
+F 0 "Q2" H 8000 3035 50  0000 C CNN
 F 1 "NTLUD4C26N" H 8000 3126 50  0000 C CNN
 F 2 "custom:UDFN6-NTLUD4" H 8000 3300 50  0001 C CNN
@@
 AR Path="/5A7C7635/5A88635F" Ref="U14"  Part="1"
 AR Path="/5A7C8234/5A88635F" Ref="U18"  Part="1"
-F 0 "U18" H 6500 5737 60  0000 C CNN
+F 0 "U6" H 6500 5737 60  0000 C CNN
 F 1 "TPS51604" H 6500 5631 60  0000 C CNN
 F 2 "custom:8-WFDFN" H 6500 5200 60  0001 C CNN
@@
 AR Path="/5A7C7635/5A886366" Ref="C28"  Part="1"
 AR Path="/5A7C8234/5A886366" Ref="C36"  Part="1"
-F 0 "C36" V 6248 5750 50  0000 C CNN
+F 0 "C12" V 6248 5750 50  0000 C CNN
 F 1 "1uF" V 6339 5750 50  0000 C CNN
 F 2 "custom:C_0402" H 6538 5600 50  0001 C CNN
@@
 AR Path="/5A7C7635/5A88636D" Ref="C27"  Part="1"
 AR Path="/5A7C8234/5A88636D" Ref="C35"  Part="1"
-F 0 "C35" V 5848 4400 50  0000 C CNN
+F 0 "C11" V 5848 4400 50  0000 C CNN
 F 1 "1uF" V 5939 4400 50  0000 C CNN
 F 2 "custom:C_0402" H 6138 4250 50  0001 C CNN
@@
 AR Path="/5A7C7635/5A886374" Ref="R24"  Part="1"
 AR Path="/5A7C8234/5A886374" Ref="R34"  Part="1"
-F 0 "R34" V 6693 4400 50  0000 C CNN
+F 0 "R4" V 6693 4400 50  0000 C CNN
 F 1 "3" V 6784 4400 50  0000 C CNN
 F 2 "custom:R_0402" V 6830 4400 50  0001 C CNN
@@
 AR Path="/5A7C7635/5A88637B" Ref="R27"  Part="1"
 AR Path="/5A7C8234/5A88637B" Ref="R37"  Part="1"
-F 0 "R37" H 8720 5596 50  0000 L CNN
+F 0 "R7" H 8720 5596 50  0000 L CNN
 F 1 "10k" H 8720 5505 50  0000 L CNN
 F 2 "custom:R_0402" V 8580 5550 50  0001 C CNN
@@
 AR Path="/5A7C7635/5A886382" Ref="R30"  Part="1"
 AR Path="/5A7C8234/5A886382" Ref="R40"  Part="1"
-F 0 "R40" H 8970 5346 50  0000 L CNN
+F 0 "R10" H 8970 5346 50  0000 L CNN
 F 1 "100k" H 8970 5255 50  0000 L CNN
 F 2 "custom:R_0402" V 8830 5300 50  0001 C CNN
@@
 AR Path="/5A7C7635/5A88638A" Ref="P14"  Part="1"
 AR Path="/5A7C8234/5A88638A" Ref="P18"  Part="1"
-F 0 "P18" H 9478 5050 60  0000 L CNN
+F 0 "P6" H 9478 5050 60  0000 L CNN
 F 1 "Pad" H 9350 4800 60  0001 C CNN
 F 2 "custom:PhasePad" H 9350 5050 60  0001 C CNN
@@
 AR Path="/5A7C7635/5A8863BF" Ref="Q9"  Part="1"
 AR Path="/5A7C8234/5A8863BF" Ref="Q12"  Part="1"
-F 0 "Q12" H 8050 4835 50  0000 C CNN
+F 0 "Q3" H 8050 4835 50  0000 C CNN
 F 1 "NTLUD4C26N" H 8050 4926 50  0000 C CNN
 F 2 "custom:UDFN6-NTLUD4" H 8050 5100 50  0001 C CNN
@@
 AR Path="/5A7C7635/5A8AFC0C" Ref="P21"  Part="1"
 AR Path="/5A7C8234/5A8AFC0C" Ref="P22"  Part="1"
-F 0 "P22" H 10528 1650 60  0000 L CNN
+F 0 "P19" H 10528 1650 60  0000 L CNN
 F 1 "Pad" H 10400 1400 60  0001 C CNN
 F 2 "custom:HOLE" H 10400 1650 60  0001 C CNN
@@
 AR Path="/5A7C7635/5AA675BC" Ref="R47"  Part="1"
 AR Path="/5A7C8234/5AA675BC" Ref="R50"  Part="1"
-F 0 "R50" H 8870 2246 50  0000 L CNN
+F 0 "R41" H 8870 2246 50  0000 L CNN
 F 1 "10k" H 8870 2155 50  0000 L CNN
 F 2 "custom:R_0402" V 8730 2200 50  0001 C CNN
@@
 AR Path="/5A7C7635/5AA8C48C" Ref="R48"  Part="1"
 AR Path="/5A7C8234/5AA8C48C" Ref="R51"  Part="1"
-F 0 "R51" H 8920 4046 50  0000 L CNN
+F 0 "R42" H 8920 4046 50  0000 L CNN
 F 1 "10k" H 8920 3955 50  0000 L CNN
 F 2 "custom:R_0402" V 8780 4000 50  0001 C CNN
@@
 AR Path="/5A7C7635/5AAB1C91" Ref="R49"  Part="1"
 AR Path="/5A7C8234/5AAB1C91" Ref="R52"  Part="1"
-F 0 "R52" H 8970 5846 50  0000 L CNN
+F 0 "R43" H 8970 5846 50  0000 L CNN
 F 1 "10k" H 8970 5755 50  0000 L CNN
 F 2 "custom:R_0402" V 8830 5800 50  0001 C CNN
@@
 Text Label 6300 4400 0    50   ~ 0
 BST_A
+$Comp
+L 6sESC:Pad P24
+U 1 1 5C39FB60
+P 3700 2300
+AR Path="/5A7E1D64/5C39FB60" Ref="P24"  Part="1"
+AR Path="/5A7C60B8/5C39FB60" Ref="P26"  Part="1"
+AR Path="/5A7C7635/5C39FB60" Ref="P28"  Part="1"
+AR Path="/5A7C8234/5C39FB60" Ref="P30"  Part="1"
+F 0 "P24" H 3828 2300 60  0000 L CNN
+F 1 "Pad" H 3700 2050 60  0001 C CNN
+F 2 "custom:FlashPad" H 3700 2300 60  0001 C CNN
+F 3 "" H 3700 2300 60  0001 C CNN
+	1    3700 2300
+	1    0    0    -1
+$EndComp
+Wire Wire Line
+	3500 2300 3350 2300
+Connection ~ 3350 2300
+Wire Wire Line
+	3350 2300 3350 2550
+$Comp
+L 6sESC:Pad P23
+U 1 1 5C3A7C3C
+P 3250 1500
+AR Path="/5A7E1D64/5C3A7C3C" Ref="P23"  Part="1"
+AR Path="/5A7C60B8/5C3A7C3C" Ref="P25"  Part="1"
+AR Path="/5A7C7635/5C3A7C3C" Ref="P27"  Part="1"
+AR Path="/5A7C8234/5C3A7C3C" Ref="P29"  Part="1"
+F 0 "P23" V 3194 1372 60  0000 R CNN
+F 1 "Pad" H 3250 1250 60  0001 C CNN
+F 2 "custom:FlashPad" H 3250 1500 60  0001 C CNN
+F 3 "" H 3250 1500 60  0001 C CNN
+	1    3250 1500
+	0    -1   -1   0
+$EndComp
+Wire Wire Line
+	3250 2550 3250 1700
 $EndSCHEMATC

Commit message: cleaning up for public
Parts:
- R2, R3, R4: value 3 -> 1
Changed lines of the file:
@@
 AR Path="/5A7C8234/5A8007E3" Ref="R32"  Part="1"
 F 0 "R2" V 6593 800 50  0000 C CNN
-F 1 "3" V 6684 800 50  0000 C CNN
+F 1 "1" V 6684 800 50  0000 C CNN
 F 2 "custom:R_0402" V 6730 800 50  0001 C CNN
 F 3 "" H 6800 800 50  0000 C CNN
@@
 AR Path="/5A7C8234/5A882B83" Ref="R33"  Part="1"
 F 0 "R3" V 6643 2600 50  0000 C CNN
-F 1 "3" V 6734 2600 50  0000 C CNN
+F 1 "1" V 6734 2600 50  0000 C CNN
 F 2 "custom:R_0402" V 6780 2600 50  0001 C CNN
 F 3 "" H 6850 2600 50  0000 C CNN
@@
 AR Path="/5A7C8234/5A886374" Ref="R34"  Part="1"
 F 0 "R4" V 6693 4400 50  0000 C CNN
-F 1 "3" V 6784 4400 50  0000 C CNN
+F 1 "1" V 6784 4400 50  0000 C CNN
 F 2 "custom:R_0402" V 6830 4400 50  0001 C CNN
 F 3 "" H 6900 4400 50  0000 C CNN
